File: LightWalker.sch (EAGLE design)
At the start: 35 parts, among them IC1 74HCT245N

Commit message: initial schema for pcb
Parts:
- C1: value 1000uf -> 0.1uf
- C2: value 0.1uf -> 1000uf
- R12, R13, R14, R15, R16, R17, R18, R19: value 10k -> 100
- R2, R3, R4, R5, R6, R7, R8, R9: value 100 -> 10k
- renumbered BLUEFRUIT_EZLINK to BLUETOOTH, I2CMULTIPLEX to I2CMULTI1, MAX9814_MIC to MIC
Connections:
- net +3V3: now also R2.1, R3.1, R4.1, R5.1, R6.1, R7.1, R8.1, R9.1; no longer R12.1, R13.1, R14.1, R15.1, R16.1, R17.1, R18.1, R19.1
- net +5V: now also C2.+; no longer C1.+
- net CS0: now also R12.1; no longer R2.1
- net CS1: now also R14.1; no longer R4.1
- net CS2: now also R16.1; no longer R6.1
- net CS3: now also R18.1; no longer R8.1
- net DATA0: now also R13.1; no longer R3.1
- net DATA1: now also R15.1; no longer R5.1
- net DATA2: now also R17.1; no longer R7.1
- net DATA3: now also R19.1; no longer R9.1
- net MIC_OUT: now also C1.+; no longer C2.+
- net N$1: now also R12.2; no longer R2.2
- net N$3: now also R13.2; no longer R3.2
- net N$4: now also R14.2; no longer R4.2
- net N$5: now also R15.2; no longer R5.2
- net N$6: now also R16.2; no longer R6.2
- net N$7: now also R17.2; no longer R7.2
- net N$8: now also R18.2; no longer R8.2
- net N$9: now also R19.2; no longer R9.2
- net SCL: now also R10.2; no longer R18.2
- net SCL0: now also R3.2; no longer R12.2
- net SCL1: now also R5.2; no longer R10.2
- net SCL2: now also R7.2; no longer R15.2
- net SCL3: now also R9.2; no longer R17.2
- net SDA: now also R11.2; no longer R19.2
- net SDA0: now also R2.2; no longer R13.2
- net SDA1: now also R4.2; no longer R11.2
- net SDA2: now also R6.2; no longer R14.2
- net SDA3: now also R8.2; no longer R16.2
Other:
- moved on the sheet: C1, C2, R10, R11, R12, R13, R14, R15, R16, R17, R18, R19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

Commit message: LightWalker board 3.0, march 2016. printed.
Parts:
- removed BLUETOOTH: (no value), pinhead:PINHD-1X7
- removed C1: 0.1uf, rcl:CPOL-USE3.5-8
- removed MIC: (no value), pinhead:PINHD-1X5
- added BLUEFRUIT1: BLUEFRUIT_EZLINK, minty:BLUEFRUIT_EZLINK
- added C4: 0.1uf, rcl:CPOL-USE5-5
- added MAX9814MIC: MAX9814MIC, minty:MAX9814MIC
Connections:
- net +3V3: now also BLUEFRUIT1.VIN, MAX9814MIC.VDD; no longer BLUETOOTH.4, MIC.2
- net AR: now also BRAINS.14/A0, MAX9814MIC.AR; no longer BRAINS.15/A1, MIC.5
- net BT_STATUS: now also BLUEFRUIT1.STS; no longer BLUETOOTH.7
- net CS1: now also LED_R_ARM.2; no longer LED_L_ARM.2
- net CS2: now also LED_L_ARM.2; no longer LED_R_ARM.2
- net DATA1: now also LED_R_ARM.1; no longer LED_L_ARM.1
- net DATA2: now also LED_L_ARM.1; no longer LED_R_ARM.1
- net GAIN: now also BRAINS.16/A2, MAX9814MIC.GAIN; no longer BRAINS.14/A0, MIC.3
- net GND: now also BLUEFRUIT1.GND, C4.-, MAX9814MIC.GND; no longer BLUETOOTH.6, C1.-, MIC.1
- net MIC_OUT: now also BRAINS.15/A1, C4.+, MAX9814MIC.OUT; no longer BRAINS.16/A2, C1.+, MIC.4
- net RX: now also BLUEFRUIT1.TX; no longer BLUETOOTH.3
- net SCL0: now also LAX.3; no longer LLX.3
- net SCL1: now also RAX.3; no longer RLX.3
- net SCL2: now also RLX.3; no longer LAX.3
- net SCL3: now also LLX.3; no longer RAX.3
- net SDA0: now also LAX.4; no longer LLX.4
- net SDA1: now also RAX.4; no longer RLX.4
- net SDA2: now also RLX.4; no longer LAX.4
- net SDA3: now also LLX.4; no longer RAX.4
- net TX: now also BLUEFRUIT1.RX; no longer BLUETOOTH.2
Other:
- moved on the sheet: LAX, LED_L_ARM, LED_R_ARM, LLX, RAX, RLX

Commit message: lightwalker PCB 4.0
Parts:
- removed 5V_IN: (no value), pinhead:PINHD-1X2
- removed BLUEFRUIT1: BLUEFRUIT_EZLINK, minty:BLUEFRUIT_EZLINK
- removed BRAINS: TEENSY_3.0_BASIC, Teensy3.0:TEENSY_3.0_BASIC
- removed C4: 0.1uf, rcl:CPOL-USE5-5
- removed LED_HORNS, LED_LEGS, LED_L_ARM, LED_R_ARM: (no value), pinhead:PINHD-1X4
- removed MAX9814MIC: MAX9814MIC, minty:MAX9814MIC
- removed R17, R18, R19: 100, resistor:R-US_0207/10
- added BRAIN: TEENSY_3.6_DIL, Teensy3.0:TEENSY_3.6_DIL
- added C3: 0.1uf, cap-master.rpt:CP-3225
- added LED_H, LED_LA, LED_LL, LED_RA, LED_RL: 2.54MM_TERMINAL_BLOCK-3, minty:2.54MM_TERMINAL_BLOCK-3
- added POWER: 2.54MM_TERMINAL_BLOCK-2, minty:2.54MM_TERMINAL_BLOCK-2
- added U$1: BLUEFRUIT_BLE_UART_FRIENDALL, minty:BLUEFRUIT_BLE_UART_FRIENDALL
- added U$4: MAX9814MICALL, minty:MAX9814MICALL
- added U1: TSR_1-2450, _traco_tsr-1:TSR_1-2450
- C2: device rcl:CPOL-USE3.5-8 -> cap-master:CP-SV-K
- LAX, LLX, RAX, RLX: value (none) -> 2.54MM_TERMINAL_BLOCK-4; device pinhead:PINHD-1X4 -> minty:2.54MM_TERMINAL_BLOCK-4
- R1, R10, R11, R12, R13, R14, R15, R16, R2, R3, R4, R5, R6, R7, R8, R9: device resistor:R-US_0207/10 -> resistor:R-US_R1206
Connections:
- removed net BT_STATUS: BLUEFRUIT1.STS, BRAINS.2
- removed net CS0: LED_HORNS.2, R12.1
- removed net CS1: LED_R_ARM.2, R14.1
- removed net CS2: LED_L_ARM.2, R16.1
- removed net CS3: LED_LEGS.2, R18.1
- removed net DATA0: LED_HORNS.1, R13.1
- removed net DATA1: LED_R_ARM.1, R15.1
- removed net DATA2: LED_L_ARM.1, R17.1
- removed net DATA3: LED_LEGS.1, R19.1
- removed net N$14: BRAINS.7, IC1A.A5
- removed net N$15: BRAINS.8, IC1A.A4
- removed net N$16: BRAINS.9, IC1A.A3
- removed net N$17: BRAINS.10, IC1A.A2
- removed net N$18: BRAINS.11, IC1A.A1
- removed net N$4: IC1A.B6, R14.2
- removed net N$7: IC1A.B3, R17.2
- removed net N$8: IC1A.B2, R18.2
- removed net N$9 (its old number): IC1A.B1, R19.2
- new net 12V: C2.+, LED_H.1, LED_LA.1, LED_LL.1, LED_RA.1, LED_RL.1, POWER.1, U1.VI
- new net 20: BRAIN.20/A6/PWM, IC1A.A6
- new net 21: BRAIN.21/A7/PWM, IC1A.A7
- new net LED_DATA_0: LED_LA.3, R12.1
- new net LED_DATA_1: LED_LL.3, R16.1
- new net LED_DATA_2: LED_RL.3, R14.1
- new net LED_DATA_3: LED_RA.3, R15.1
- new net LED_DATA_4: LED_H.3, R13.1
- new net N$1: BRAIN.2/PWM, IC1A.A8
- new net N$12: IC1A.B2, R15.2
- new net N$2: BRAIN.5/PWM, IC1A.A5
- new net PIN14: BRAIN.14/A0/PWM, IC1A.A1
- net +3V3: now also BRAIN.3.3V, LAX.4, LLX.4, RAX.4, RLX.4, U$1.VIN, U$4.VDD; no longer BLUEFRUIT1.VIN, BRAINS.3.3V, LAX.1, LLX.1, MAX9814MIC.VDD, RAX.1, RLX.1
- net +5V: now also BRAIN.VIN, U1.VO; no longer 5V_IN.1, BRAINS.VIN, C2.+, LED_HORNS.4, LED_LEGS.4, LED_L_ARM.4, LED_R_ARM.4
- net AR: now also BRAIN.23/A9/T/PWM, U$4.AR; no longer BRAINS.14/A0, MAX9814MIC.AR
- net GAIN: now also BRAIN.19/A5/T/SCL0, U$4.GAIN; no longer BRAINS.16/A2, MAX9814MIC.GAIN
- net GND: now also BRAIN.GND, C3.-, LAX.3, LED_H.2, LED_LA.2, LED_LL.2, LED_RA.2, LED_RL.2, LLX.3, POWER.2, RAX.3, RLX.3, U$1.CTS, U$1.GND, U$4.GND, U1.GND; no longer 5V_IN.2, BLUEFRUIT1.GND, BRAINS.GND, C4.-, LAX.2, LED_HORNS.3, LED_LEGS.3, LED_L_ARM.3, LED_R_ARM.3, LLX.2, MAX9814MIC.GND, RAX.2, RLX.2
- net MIC_OUT: now also BRAIN.22/A8/T/PWM, C3.+, U$4.OUT; no longer BRAINS.15/A1, C4.+, MAX9814MIC.OUT
- net N$10: now also IC1A.B4, R13.2; no longer BRAINS.4, IC1A.A8
- net N$11: now also IC1A.B3, R14.2; no longer BRAINS.5, IC1A.A7
- net N$13: now also IC1A.B1, R16.2; no longer BRAINS.6, IC1A.A6
- net N$3: now also BRAIN.6/PWM, IC1A.A4; no longer IC1A.B7, R13.2
- net N$5: now also BRAIN.7/RX3/PWM, IC1A.A3; no longer IC1A.B5, R15.2
- net N$6: now also BRAIN.8/TX3/PWM, IC1A.A2; no longer IC1A.B4, R16.2
- net RX: now also BRAIN.31/A12/RX4, U$1.TXO; no longer BLUEFRUIT1.TX, BRAINS.0
- net SCL: now also BRAIN.37/A18/SCL1/PWM; no longer BRAINS.19/A5
- net SCL0: now also LAX.2; no longer LAX.3
- net SCL1: now also RAX.2; no longer RAX.3
- net SCL2: now also RLX.2; no longer RLX.3
- net SCL3: now also LLX.2; no longer LLX.3
- net SDA: now also BRAIN.38/A19/SDA1/PWM; no longer BRAINS.18/A4
- net SDA0: now also LAX.1; no longer LAX.4
- net SDA1: now also RAX.1; no longer RAX.4
- net SDA2: now also RLX.1; no longer RLX.4
- net SDA3: now also LLX.1; no longer LLX.4
- net TX: now also BRAIN.32/A13/TX4, U$1.RXI; no longer BLUEFRUIT1.RX, BRAINS.1
Other:
- note added: "4.0_a_sep2018"
- note removed: "3.0_a_march2016"
- moved on the sheet: C2, IC1, IC1P, R12, R13, R14, R15, R16
